Commit message: Deleted Unused files. changes in pelican URDF.

File: rotors_description/urdf/pelican.xacro (robot description, xacro)
@@ -19,4 +19,5 @@
   <!-- Properties  -->
   <!-- TODO(ff): Update these params when identifying the model. -->
+  <!-- SIA: Changed max velocity, rolling moment coeff and time constants.-->
   <xacro:property name="namespace" value="$(arg namespace)" />
   <xacro:property name="rotor_velocity_slowdown_sim" value="10" />
@@ -32,9 +33,9 @@
   <xacro:property name="motor_constant" value="9.9865e-06" /> <!-- [kg m/s^2] -->
   <xacro:property name="moment_constant" value="0.016" /> <!-- [m] -->
-  <xacro:property name="time_constant_up" value="0.0125" /> <!-- [s] -->
-  <xacro:property name="time_constant_down" value="0.025" /> <!-- [s] -->
-  <xacro:property name="max_rot_velocity" value="838" /> <!-- [rad/s] -->
+  <xacro:property name="time_constant_up" value="0.0005" /> <!-- [s] -->
+  <xacro:property name="time_constant_down" value="0.005" /> <!-- [s] -->
+  <xacro:property name="max_rot_velocity" value="1000" /> <!-- [rad/s] -->
   <xacro:property name="rotor_drag_coefficient" value="8.06428e-05" />
-  <xacro:property name="rolling_moment_coefficient" value="0.000001" />
+  <xacro:property name="rolling_moment_coefficient" value="0.00000" />
   <!-- Property Blocks -->
   <xacro:property name="body_inertia">

Commit message: fixed yaw control problem.

File: rotors_description/urdf/pelican.xacro (robot description, xacro)
@@ -35,7 +35,7 @@
   <xacro:property name="time_constant_up" value="0.0005" /> <!-- [s] -->
   <xacro:property name="time_constant_down" value="0.005" /> <!-- [s] -->
-  <xacro:property name="max_rot_velocity" value="1000" /> <!-- [rad/s] -->
+  <xacro:property name="max_rot_velocity" value="838" /> <!-- [rad/s] -->
   <xacro:property name="rotor_drag_coefficient" value="8.06428e-05" />
-  <xacro:property name="rolling_moment_coefficient" value="0.00000" />
+  <xacro:property name="rolling_moment_coefficient" value="0.000001" />
   <!-- Property Blocks -->
   <xacro:property name="body_inertia">
